File: GETOU_.kicad_pcb (KiCad board)
At the start: 2 copper layers, 1 part

Commit message: Modify PCB
Parts:
- removed A1: RaspberryPi_Pico, Module:RaspberryPi_Pico_Common_Unspecified
- added D1: 1N4148, Diode_THT:D_DO-35_SOD27_P7.62mm_Horizontal, F.Cu at (90.2, 68.4)
- added D10: 1N4148, Diode_THT:D_DO-35_SOD27_P7.62mm_Horizontal, F.Cu at (90.2, 100.3)
- added D11: 1N4148, Diode_THT:D_DO-35_SOD27_P7.62mm_Horizontal, F.Cu at (90.2, 103.9)
- added D12: 1N4148, Diode_THT:D_DO-35_SOD27_P7.62mm_Horizontal, F.Cu at (90.2, 107.5)
- added D2: 1N4148, Diode_THT:D_DO-35_SOD27_P7.62mm_Horizontal, F.Cu at (90.2, 72.0)
- added D3: 1N4148, Diode_THT:D_DO-35_SOD27_P7.62mm_Horizontal, F.Cu at (90.2, 75.5)
- added D4: 1N4148, Diode_THT:D_DO-35_SOD27_P7.62mm_Horizontal, F.Cu at (90.2, 79.0)
- added D5: 1N4148, Diode_THT:D_DO-35_SOD27_P7.62mm_Horizontal, F.Cu at (90.2, 82.6)
- added D6: 1N4148, Diode_THT:D_DO-35_SOD27_P7.62mm_Horizontal, F.Cu at (90.2, 86.2)
- added D7: 1N4148, Diode_THT:D_DO-35_SOD27_P7.62mm_Horizontal, F.Cu at (90.2, 89.7)
- added D8: 1N4148, Diode_THT:D_DO-35_SOD27_P7.62mm_Horizontal, F.Cu at (90.2, 93.2)
- added D9: 1N4148, Diode_THT:D_DO-35_SOD27_P7.62mm_Horizontal, F.Cu at (90.2, 96.8)
- added S1: MX1A-11NN, footprints:SW_MX1A-11NN, F.Cu at (110.0, 69.4)
- added S10: MX1A-11NN, footprints:SW_MX1A-11NN, F.Cu at (161.1, 69.4)
- added S11: MX1A-11NN, footprints:SW_MX1A-11NN, F.Cu at (161.1, 86.5)
- added S12: MX1A-11NN, footprints:SW_MX1A-11NN, F.Cu at (161.1, 103.5)
- added S2: MX1A-11NN, footprints:SW_MX1A-11NN, F.Cu at (110.0, 86.5)
- added S3: MX1A-11NN, footprints:SW_MX1A-11NN, F.Cu at (110.0, 103.5)
- added S4: MX1A-11NN, footprints:SW_MX1A-11NN, F.Cu at (127.0, 69.4)
- added S5: MX1A-11NN, footprints:SW_MX1A-11NN, F.Cu at (127.0, 86.5)
- added S6: MX1A-11NN, footprints:SW_MX1A-11NN, F.Cu at (127.0, 103.5)
- added S7: MX1A-11NN, footprints:SW_MX1A-11NN, F.Cu at (144.0, 69.4)
- added S8: MX1A-11NN, footprints:SW_MX1A-11NN, F.Cu at (144.0, 86.5)
- added S9: MX1A-11NN, footprints:SW_MX1A-11NN, F.Cu at (144.0, 103.5)
- added U1: XIAO-RP2040-DIP, footprints:XIAO-RP2040-DIP, F.Cu at (180.0, 87.0)
Routing:
- net col0: track 0.00 -> 149.0 mm
- net col1: track 0.00 -> 124.5 mm, vias 0 -> 1
- net row0: track 0.00 -> 120.5 mm
- net col2: track 0.00 -> 117.8 mm
- net col3: track 0.00 -> 106.2 mm
- net row1: track 0.00 -> 98.8 mm, vias 0 -> 1
- net Net-(D11-A): track 0.00 -> 96.5 mm, vias 0 -> 1
- net Net-(D10-A): track 0.00 -> 83.5 mm, vias 0 -> 1
- net Net-(D7-A): track 0.00 -> 78.8 mm, vias 0 -> 1
- net row2: track 0.00 -> 73.6 mm
- net Net-(D9-A): track 0.00 -> 67.8 mm, vias 0 -> 1
- net Net-(D8-A): track 0.00 -> 53.7 mm
- net Net-(D12-A): track 0.00 -> 52.5 mm
- net Net-(D6-A): track 0.00 -> 42.9 mm, vias 0 -> 1
- net Net-(D4-A): track 0.00 -> 42.4 mm, vias 0 -> 1
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Other:
- board outline added: 106.5 x 58 mm
