File: GETOU_.kicad_sch (KiCad schematic)
At the start: 0 parts

Commit message: Add KB switches and RPI Pico
Parts:
- added A1: RaspberryPi_Pico, Module:RaspberryPi_Pico_Common_Unspecified, symbol MCU_Module:RaspberryPi_Pico
- added S1, S10, S11, S12, S13, S14, S15, S16, S17, S18, S19, S2, S20, S21, S22, S23, S24, S25, S26, S27, S28, S29, S3, S30, S31, S32, S33, S34, S35, S36, S37, S38, S39, S4, S40, S41, S42, S43, S44, S45, S46, S47, S48, S49, S5, S50, S51, S52, S53, S54, S55, S56, S57, S58, S59, S6, S60, S61, S62, S63, S64, S65, S66, S67, S68, S69, S7, S70, S71, S72, S73, S74, S75, S76, S77, S78, S79, S8, S80, S81, S82, S83, S84, S85, S86, S87, S88, S9: MX1A-11NN, MX1A-11NN:SW_MX1A-11NN, symbol MX1A-11NN:MX1A-11NN
Connections:
- new net: A1.13 (GND), A1.18 (GND), A1.23 (GND), A1.28 (GND), A1.3 (GND), A1.38 (GND), A1.8 (GND)

Commit message: Modify Schematic
Parts:
- removed S13, S14, S15, S16, S17, S18, S19, S20, S21, S22, S23, S24, S25, S26, S27, S28, S29, S30, S31, S32, S33, S34, S35, S36, S37, S38, S39, S40, S41, S42, S43, S44, S45, S46, S47, S48, S49, S50, S51, S52, S53, S54, S55, S56, S57, S58, S59, S60, S61, S62, S63, S64, S65, S66, S67, S68, S69, S70, S71, S72, S73, S74, S75, S76, S77, S78, S79, S80, S81, S82, S83, S84, S85, S86, S87, S88: MX1A-11NN, MX1A-11NN:SW_MX1A-11NN, symbol MX1A-11NN:MX1A-11NN
Connections:
- net S10: now reaches S10.1
- net S10: now also A1.12 (GPIO9)
- net GND: now reaches S10.2
- net GND: now also A1.13 (GND), A1.18 (GND), A1.23 (GND), A1.28 (GND), A1.3 (GND), A1.38 (GND), A1.8 (GND), S1.2, S11.2, S12.2, S2.2, S3.2, S4.2, S5.2, S6.2, S7.2, S8.2, S9.2
- net S9: now reaches S9.1
- net S9: now also A1.11 (GPIO8)
- net S1: now reaches S1.1
- net S1: now also A1.1 (GPIO0)
- net S11: now reaches S11.1
- net S11: now also A1.14 (GPIO10)
- net S6: now reaches S6.1
- net S6: now also A1.7 (GPIO5)
- net S4: now reaches S4.1
- net S4: now also A1.5 (GPIO3)
- net S8: now reaches S8.1
- net S8: now also A1.10 (GPIO7)
- net S5: now reaches S5.1
- net S5: now also A1.6 (GPIO4)
- net S3: now reaches S3.1
- net S3: now also A1.4 (GPIO2)
- net S2: now reaches S2.1
- net S2: now also A1.2 (GPIO1)
- net S12: now reaches A1.15 (GPIO11)
- net S12: now also S12.1
- net S7: now reaches A1.9 (GPIO6)
- net S7: now also S7.1
Other:
- moved on the sheet: A1, S1, S10, S11, S12, S2, S3, S4, S5, S6, S7, S8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

Commit message: Modify PCB
Parts:
- removed A1: RaspberryPi_Pico, Module:RaspberryPi_Pico_Common_Unspecified, symbol MCU_Module:RaspberryPi_Pico
- added D1, D10, D11, D12, D2, D3, D4, D5, D6, D7, D8, D9: 1N4148, Diode_THT:D_DO-35_SOD27_P7.62mm_Horizontal, symbol Diode:1N4148
- added U1: XIAO-RP2040-DIP, footprints:XIAO-RP2040-DIP, symbol Seeed_Studio_XIAO_Series:XIAO-RP2040-DIP
- S1, S10, S11, S12, S2, S3, S4, S5, S6, S7, S8, S9: footprint MX1A-11NN:SW_MX1A-11NN -> footprints:SW_MX1A-11NN
Connections:
- net S11 is gone; now on net row2: S11.1
- net S12 is gone; now on net row2: S12.1
- net S2 is gone; now on net row0: S2.1
- net S3 is gone; now on net row0: S3.1
- net S4 is gone; now on net row0: S4.1
- net S6 is gone; now on net row1: S6.1
- net S7 is gone; now on net row1: S7.1
- net S8 is gone; now on net row1: S8.1
- net S9 is gone; now on net row2: S9.1
- removed net GND: S1.2, S10.2, S11.2, S12.2, S2.2, S3.2, S4.2, S5.2, S6.2, S7.2, S8.2, S9.2
- net S1 renamed row0
- net row0: now also U1.7 (GPIO0/TX)
- net S10 renamed row2
- net row2: now also U1.9 (GPIO2/SCK)
- net S5 renamed row1
- net row1: now also U1.8 (GPIO1/RX)
- new net: D11.2 (A), S10.2
- new net: D7.2 (A), S7.2
- new net: D12.2 (A), S9.2
- new net: D1.2 (A), S1.2
- new net: D4.2 (A), S4.2
- new net: D9.2 (A), S12.2
- new net: D8.2 (A), S8.2
- new net: D10.2 (A), S11.2
- new net: D6.2 (A), S6.2
- new net: D5.2 (A), S5.2
- new net: D3.2 (A), S3.2
- new net: D2.2 (A), S2.2
- new net col0: D1.1 (K), D12.1 (K), D5.1 (K), U1.11 (GPIO3/MOSI)
- new net col1: D11.1 (K), D2.1 (K), U1.10 (GPIO4/MISO)
- new net col2: D10.1 (K), D3.1 (K), D7.1 (K), U1.5 (GPIO6/SDA)
- new net col3: D4.1 (K), D8.1 (K), D9.1 (K), U1.6 (GPIO7/SCL)
Other:
- moved on the sheet: S1, S10, S11, S12, S2, S3, S4, S5, S6, S7, S8, S9
